Commit message: Fix Vehicle Description to AW Style

File: lomby_vehicle_description/urdf/vehicle.xacro (robot description, xacro)
@@ -8,5 +8,5 @@
       <origin xyz="${vehicle_info['/**']['ros__parameters']['wheel_base']/2.0} 0 0" rpy="${pi/2.0} 0 ${pi}"/>
       <geometry>
-        <mesh filename="package://sample_vehicle_description/mesh/lexus.dae" scale="1 1 1"/>
+        <mesh filename="package://lomby_vehicle_description/mesh/lomby.dae" scale="1 1 1"/>
       </geometry>
     </visual>

Commit message: Modify offset on X axis

File: lomby_vehicle_description/urdf/vehicle.xacro (robot description, xacro)
@@ -6,5 +6,6 @@
   <link name="base_link">
     <visual>
-      <origin xyz="${vehicle_info['/**']['ros__parameters']['wheel_base']/2.0} 0 0" rpy="${pi/2.0} 0 ${pi}"/>
+      <!-- <origin xyz="${vehicle_info['/**']['ros__parameters']['wheel_base']/2.0} 0 0" rpy="${pi/2.0} 0 ${pi}"/> -->
+      <origin xyz="0 0 0" rpy="${pi/2.0} 0 ${pi}"/>
       <geometry>
         <mesh filename="package://lomby_vehicle_description/mesh/lomby.dae" scale="1 1 1"/>

Commit message: Working Version of Vehicle Frame along with DAE and correct vehicle parameters

File: lomby_vehicle_description/urdf/vehicle.xacro (robot description, xacro)
@@ -2,10 +2,9 @@
 <robot xmlns:xacro="http://ros.org/wiki/xacro">
   <!-- load parameter -->
-  <xacro:property name="vehicle_info" value="${xacro.load_yaml('$(find sample_vehicle_description)/config/vehicle_info.param.yaml')}"/>
+  <xacro:property name="vehicle_info" value="${xacro.load_yaml('$(find lomby_vehicle_description)/config/vehicle_info.param.yaml')}"/>
   <!-- vehicle body -->
   <link name="base_link">
     <visual>
-      <!-- <origin xyz="${vehicle_info['/**']['ros__parameters']['wheel_base']/2.0} 0 0" rpy="${pi/2.0} 0 ${pi}"/> -->
-      <origin xyz="0 0 0" rpy="${pi/2.0} 0 ${pi}"/>
+      <origin xyz="${vehicle_info['/**']['ros__parameters']['wheel_base']*1.1} 0 0.15" rpy="${pi/2.0} 0 0"/>
       <geometry>
         <mesh filename="package://lomby_vehicle_description/mesh/lomby.dae" scale="1 1 1"/>
